File: elec/motor_board/motor_board.kicad_pcb (KiCad board)
At the start: 2 copper layers, 42 x 41.2 mm, 2 parts, among them J3 Conn_01x08

Commit message: Update silkscreen
Other:
- board size 42 x 41.2 mm -> 42 x 42.2 mm
- board text added: "Motor board v2.1 Tibo 27/02/2025"
- board text added: "v2.1"
- board text removed: "Motor board v2.0 Thibaut 26/01/2025"
Changed lines of the file:
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@@
 		(fp_circle
 			(center 39.25 13.5)
-			(end 42 13.5)
+			(end 42.15 13.5)
 			(stroke
 				(width 0.05)
-				(type default)
+				(type solid)
 			)
 			(fill no)
@@
 	)
 	(gr_circle
-		(center 181.75 110.75)
-		(end 183.25 110.75)
+		(center 187.5 112)
+		(end 189 112)
 		(stroke
 			(width 0.2)
@@
 	)
 	(gr_circle
-		(center 170 74)
-		(end 171.5 74)
+		(center 168.5 74)
+		(end 170 74)
 		(stroke
 			(width 0.2)
@@
 	)
 	(gr_circle
-		(center 195 74)
-		(end 196.5 74)
+		(center 196.5 74)
+		(end 198 74)
 		(stroke
 			(width 0.2)
@@
 	(gr_rect
 		(start 160.75 71.75)
-		(end 202.75 113)
+		(end 202.75 114)
 		(stroke
 			(width 0.2)
@@
 	)
 	(gr_text "B1"
-		(at 184.75 78.25 90)
+		(at 184.75 75 90)
 		(layer "F.SilkS")
 		(effects
@@
 	)
 	(gr_text "A1"
-		(at 182.75 78.25 90)
+		(at 182.75 75 90)
 		(layer "F.SilkS")
 		(effects
@@
 	)
 	(gr_text "A4"
-		(at 178.75 78.25 90)
-		(layer "F.SilkS")
-		(effects
-			(font
-				(size 1 1)
-				(thickness 0.15)
-			)
-			(justify left bottom)
-		)
-	)
-	(gr_text "Motor board v2.0\nThibaut 26/01/2025"
+		(at 178.75 75 90)
+		(layer "F.SilkS")
+		(effects
+			(font
+				(size 1 1)
+				(thickness 0.15)
+			)
+			(justify left bottom)
+		)
+	)
+	(gr_text "Motor board v2.1\nTibo 27/02/2025"
 		(at 181.5 95 0)
 		(layer "F.SilkS")
@@
 	)
 	(gr_text "A2"
-		(at 180.75 78.25 90)
+		(at 180.5 75 90)
 		(layer "F.SilkS")
 		(effects
@@
 	)
 	(gr_text "A3"
-		(at 176.75 78.25 90)
+		(at 176.75 75 90)
 		(layer "F.SilkS")
 		(effects
@@
 	)
 	(gr_text "B3"
-		(at 191 78.25 90)
+		(at 191 75 90)
 		(layer "F.SilkS")
 		(effects
@@
 	)
 	(gr_text "B4"
-		(at 188.75 78.25 90)
+		(at 188.75 75 90)
 		(layer "F.SilkS")
 		(effects
@@
 	)
 	(gr_text "B2"
-		(at 186.75 78.25 90)
+		(at 186.75 75 90)
 		(layer "F.SilkS")
 		(effects
@@
 	)
 	(gr_text "A2"
-		(at 179.75 78.25 -90)
+		(at 179.75 75 -90)
 		(layer "B.SilkS")
 		(effects
@@
 	)
 	(gr_text "B3"
-		(at 189.75 78.25 -90)
+		(at 189.75 75 -90)
 		(layer "B.SilkS")
 		(effects
@@
 	)
 	(gr_text "A1"
-		(at 181.75 78.25 -90)
+		(at 181.75 75 -90)
 		(layer "B.SilkS")
 		(effects
@@
 	)
 	(gr_text "B4"
-		(at 187.5 78.25 -90)
+		(at 187.5 75 -90)
 		(layer "B.SilkS")
 		(effects
@@
 	)
 	(gr_text "A4"
-		(at 177.75 78.25 -90)
+		(at 177.75 75 -90)
 		(layer "B.SilkS")
 		(effects
@@
 	)
 	(gr_text "B2"
-		(at 185.5 78.25 -90)
-		(layer "B.SilkS")
-		(effects
-			(font
-				(size 1 1)
-				(thickness 0.15)
-			)
-			(justify left bottom mirror)
-		)
-	)
-	(gr_text "Motor board v2.0\nThibaut 26/01/2025"
-		(at 197 94.75 -0)
+		(at 185.5 75 -90)
+		(layer "B.SilkS")
+		(effects
+			(font
+				(size 1 1)
+				(thickness 0.15)
+			)
+			(justify left bottom mirror)
+		)
+	)
+	(gr_text "Motor board v2.1\nTibo 27/02/2025"
+		(at 197 94.75 0)
 		(layer "B.SilkS")
 		(effects
@@
 	)
 	(gr_text "A3"
-		(at 175.5 78.25 -90)
+		(at 175.5 75 -90)
+		(layer "B.SilkS")
+		(effects
+			(font
+				(size 1 1)
+				(thickness 0.15)
+			)
+			(justify left bottom mirror)
+		)
+	)
+	(gr_text "v2.1"
+		(at 163 73.5 90)
 		(layer "B.SilkS")
 		(effects
@@
 	)
 	(gr_text "B1"
-		(at 183.5 78.25 -90)
-		(layer "B.SilkS")
-		(effects
+		(at 183.5 75 -90)
+		(layer "B.SilkS")
+		(effects

Commit message: Finalize PCB order
Parts:
- added J4: Conn_01x08, Connector_PinSocket_2.00mm:PinSocket_1x08_P2.00mm_Vertical, F.Cu at (190.2, 73.5)
Routing:
- net /B4: track 37.9 -> 41.6 mm
- net /B3: track 29.7 -> 33.5 mm
- net /B2: track 9.53 -> 13.3 mm
- net /B1: track 20.4 -> 24.2 mm
- net /A4: track 20.1 -> 23.9 mm
- net /A3: track 8.28 -> 12.0 mm
- net /A2: track 32.5 -> 36.3 mm
- net /A1: track 41.0 -> 44.8 mm
