File: elec/clockclock_main/motor_driver.kicad_sch (KiCad schematic)
At the start: 9 parts, among them M1 Conn motor 0, M2 Conn motor 1, U3 74HCT595, U4 VID6606

Commit message: Fix typo
Other:
- note added: "8 bits shift register"
- note removed: "8 bit shift register"
Changed lines of the file:
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@@
 		(rev "v2.1")
 	)
-	(text "8 bit shift register"
+	(text "8 bits shift register"
 		(exclude_from_sim no)
 		(at 104.394 141.478 0)
